File: AT86RF215 Breakout Board.kicad_pcb (KiCad board)
At the start: 4 copper layers, 75 x 50 mm, 54 parts, among them J1 USB_C, J2 896 ISM, J3 GPIO, J4 2.4G ISM, J5 Molex 53748-0408, J6 Frontend GPIO, J7 SPI Header, U1 XC6206P332MR-G, U2 AT86RF215, X1 7L26002007

Commit message: Add files via upload
Other:
- board text added: "Controlled Impedance Board JLC04161H-3313 Stackup"
Changed lines of the file:
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@@
+		)
+	)
+	(gr_text "Controlled Impedance Board\nJLC04161H-3313 Stackup"
+		(at 138.35 31.55 0)
+		(layer "F.Fab")
+		(effects
+			(font
+				(size 2 2)
+				(thickness 0.15)
+			)
+			(justify bottom)
 		)
 	)

Commit message: added local symbol and footprint libs
Parts:
- B1, B2: footprint U's Footprint Library:0896BM15E0025 -> Library:0896BM15E0025
- C1, C10, C11, C12, C13, C14, C15, C16, C17, C18, C19, C2, C20, C21, C22, C3, C4, C5, C6, C7, C8, C9: footprint Capacitor_SMD:C_0402_1005Metric -> Library:C_0402_1005Metric
- G*** (x2): footprint LOGO -> Library:LOGO
- H1, H2, H3, H4: footprint MountingHole:MountingHole_3.2mm_M3_ISO14580 -> Library:MountingHole_3.2mm_M3_ISO14580
- J1: footprint Connector_USB:USB_C_Receptacle_GCT_USB4125-xx-x-0190_6P_TopMnt_Horizontal -> Library:USB_C_Receptacle_GCT_USB4125-xx-x-0190_6P_TopMnt_Horizontal
- J2, J4: footprint U's Footprint Library:BWSMA-KE-Z001 -> Library:BWSMA-KE-Z001
- J3, J6, J7: footprint Connector_PinHeader_2.54mm:PinHeader_1x06_P2.54mm_Vertical -> Library:PinHeader_1x06_P2.54mm_Vertical
- J5: footprint Connector_Molex:Molex_SlimStack_53748-0408_2x20_P0.50mm_Vertical -> Library:Molex_SlimStack_53748-0408_2x20_P0.50mm_Vertical
- JP1: footprint Jumper:SolderJumper-2_P1.3mm_Bridged_RoundedPad1.0x1.5mm -> Library:SolderJumper-2_P1.3mm_Bridged_RoundedPad1.0x1.5mm
- L1: footprint Inductor_SMD:L_0402_1005Metric -> Library:L_0402_1005Metric
- R1, R2, R3, R4, R5, R6, R7: footprint Resistor_SMD:R_0603_1608Metric -> Library:R_0603_1608Metric
- TP1, TP2, TP4, TP5: footprint TestPoint:TestPoint_Pad_D1.0mm -> Library:TestPoint_Pad_D1.0mm
- TP3: footprint Connector_PinHeader_2.54mm:PinHeader_1x02_P2.54mm_Vertical -> Library:PinHeader_1x02_P2.54mm_Vertical
- U1: footprint Package_TO_SOT_SMD:SOT-23-3 -> Library:SOT-23-3
- U2: footprint U's Footprint Library:AT86RF215 -> Library:AT86RF215
- X1: footprint U's Footprint Library:7L26002007 -> Library:7L26002007
Changed lines of the file:
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@@
 	(net 44 "/CLKO_conn")
 	(net 45 "/~{RST}_conn")
-	(footprint "Connector_USB:USB_C_Receptacle_GCT_USB4125-xx-x-0190_6P_TopMnt_Horizontal"
+	(footprint "Library:USB_C_Receptacle_GCT_USB4125-xx-x-0190_6P_TopMnt_Horizontal"
 		(locked yes)
 		(layer "F.Cu")
@@
 		)
 	)
-	(footprint "Capacitor_SMD:C_0402_1005Metric"
+	(footprint "Library:C_0402_1005Metric"
 		(locked yes)
 		(layer "F.Cu")
@@
 		)
 	)
-	(footprint "Capacitor_SMD:C_0402_1005Metric"
+	(footprint "Library:C_0402_1005Metric"
 		(locked yes)
 		(layer "F.Cu")
@@
 		)
 	)
-	(footprint "Resistor_SMD:R_0603_1608Metric"
+	(footprint "Library:R_0603_1608Metric"
 		(locked yes)
 		(layer "F.Cu")
@@
 		)
 	)
-	(footprint "MountingHole:MountingHole_3.2mm_M3_ISO14580"
+	(footprint "Library:MountingHole_3.2mm_M3_ISO14580"
 		(locked yes)
 		(layer "F.Cu")
@@
 		)
 	)
-	(footprint "Capacitor_SMD:C_0402_1005Metric"
+	(footprint "Library:C_0402_1005Metric"
 		(locked yes)
 		(layer "F.Cu")
@@
 		)
 	)
-	(footprint "Capacitor_SMD:C_0402_1005Metric"
+	(footprint "Library:C_0402_1005Metric"
 		(locked yes)
 		(layer "F.Cu")
@@
 		)
 	)
-	(footprint "TestPoint:TestPoint_Pad_D1.0mm"
+	(footprint "Library:TestPoint_Pad_D1.0mm"
 		(locked yes)
 		(layer "F.Cu")
@@
 		)
 	)
-	(footprint "U's Footprint Library:BWSMA-KE-Z001"
+	(footprint "Library:BWSMA-KE-Z001"
 		(locked yes)
 		(layer "F.Cu")
@@
 		)
 	)
-	(footprint "U's Footprint Library:0896BM15E0025"
+	(footprint "Library:0896BM15E0025"
 		(locked yes)
 		(layer "F.Cu")
@@
 		)
 	)
-	(footprint "Resistor_SMD:R_0603_1608Metric"
+	(footprint "Library:R_0603_1608Metric"
 		(locked yes)
 		(layer "F.Cu")
@@
 		)
 	)
-	(footprint "MountingHole:MountingHole_3.2mm_M3_ISO14580"
+	(footprint "Library:MountingHole_3.2mm_M3_ISO14580"
 		(locked yes)
 		(layer "F.Cu")
@@
 		)
 	)
-	(footprint "Capacitor_SMD:C_0402_1005Metric"
+	(footprint "Library:C_0402_1005Metric"
 		(locked yes)
 		(layer "F.Cu")
@@
 		)
 	)
-	(footprint "Capacitor_SMD:C_0402_1005Metric"
+	(footprint "Library:C_0402_1005Metric"
 		(locked yes)
 		(layer "F.Cu")
@@
 		)
 	)
-	(footprint "TestPoint:TestPoint_Pad_D1.0mm"
+	(footprint "Library:TestPoint_Pad_D1.0mm"
 		(locked yes)
 		(layer "F.Cu")
@@
 		)
 	)
-	(footprint "Connector_PinHeader_2.54mm:PinHeader_1x02_P2.54mm_Vertical"
+	(footprint "Library:PinHeader_1x02_P2.54mm_Vertical"
 		(locked yes)
 		(layer "F.Cu")
@@
 		)
 	)
-	(footprint "Inductor_SMD:L_0402_1005Metric"
+	(footprint "Library:L_0402_1005Metric"
 		(locked yes)
 		(layer "F.Cu")
@@
 		)
 	)
-	(footprint "Capacitor_SMD:C_0402_1005Metric"
+	(footprint "Library:C_0402_1005Metric"
 		(locked yes)
 		(layer "F.Cu")
@@
 		)
 	)
-	(footprint "U's Footprint Library:7L26002007"
+	(footprint "Library:7L26002007"
 		(locked yes)
 		(layer "F.Cu")
@@
 		)
 	)
-	(footprint "Capacitor_SMD:C_0402_1005Metric"
+	(footprint "Library:C_0402_1005Metric"
 		(locked yes)
 		(layer "F.Cu")
@@
 		)
 	)
-	(footprint "Jumper:SolderJumper-2_P1.3mm_Bridged_RoundedPad1.0x1.5mm"
+	(footprint "Library:SolderJumper-2_P1.3mm_Bridged_RoundedPad1.0x1.5mm"
 		(locked yes)
 		(layer "F.Cu")
@@
 		)
 	)
-	(footprint "Connector_Molex:Molex_SlimStack_53748-0408_2x20_P0.50mm_Vertical"
+	(footprint "Library:Molex_SlimStack_53748-0408_2x20_P0.50mm_Vertical"
 		(locked yes)
 		(layer "F.Cu")
@@
 		)
 	)
-	(footprint "U's Footprint Library:BWSMA-KE-Z001"
+	(footprint "Library:BWSMA-KE-Z001"
 		(locked yes)
 		(layer "F.Cu")
@@
 		)
 	)
-	(footprint "Connector_PinHeader_2.54mm:PinHeader_1x06_P2.54mm_Vertical"
+	(footprint "Library:PinHeader_1x06_P2.54mm_Vertical"
 		(locked yes)
 		(layer "F.Cu")
@@
 		)
 	)
-	(footprint "U's Footprint Library:AT86RF215"
+	(footprint "Library:AT86RF215"
 		(locked yes)
 		(layer "F.Cu")
@@
 		)
 	)
-	(footprint "MountingHole:MountingHole_3.2mm_M3_ISO14580"
+	(footprint "Library:MountingHole_3.2mm_M3_ISO14580"
 		(locked yes)
 		(layer "F.Cu")
@@
 		)
 	)
-	(footprint "Resistor_SMD:R_0603_1608Metric"
+	(footprint "Library:R_0603_1608Metric"
 		(locked yes)
 		(layer "F.Cu")
@@
 		)
 	)
-	(footprint "Connector_PinHeader_2.54mm:PinHeader_1x06_P2.54mm_Vertical"
+	(footprint "Library:PinHeader_1x06_P2.54mm_Vertical"
 		(locked yes)
 		(layer "F.Cu")
@@
 		)
 	)
-	(footprint "LOGO"
+	(footprint "Library:LOGO"
 		(locked yes)
 		(layer "F.Cu")
@@
 		)
 	)
-	(footprint "Connector_PinHeader_2.54mm:PinHeader_1x06_P2.54mm_Vertical"
+	(footprint "Library:PinHeader_1x06_P2.54mm_Vertical"
 		(locked yes)
 		(layer "F.Cu")
@@
 		)
 	)
-	(footprint "MountingHole:MountingHole_3.2mm_M3_ISO14580"
+	(footprint "Library:MountingHole_3.2mm_M3_ISO14580"
 		(locked yes)
 		(layer "F.Cu")
@@
 		)
 	)
-	(footprint "Capacitor_SMD:C_0402_1005Metric"
+	(footprint "Library:C_0402_1005Metric"
 		(locked yes)
 		(layer "F.Cu")
@@
 		)
 	)
-	(footprint "Capacitor_SMD:C_0402_1005Metric"
+	(footprint "Library:C_0402_1005Metric"
 		(locked yes)
 		(layer "F.Cu")
@@
 		)
 	)
-	(footprint "Resistor_SMD:R_0603_1608Metric"
+	(footprint "Library:R_0603_1608Metric"
 		(locked yes)
 		(layer "F.Cu")
@@
 		)
 	)
-	(footprint "Capacitor_SMD:C_0402_1005Metric"
+	(footprint "Library:C_0402_1005Metric"
 		(locked yes)
 		(layer "F.Cu")
@@
 		)
 	)
-	(footprint "Capacitor_SMD:C_0402_1005Metric"
+	(footprint "Library:C_0402_1005Metric"
 		(locked yes)
 		(layer "F.Cu")
@@
 		)
 	)
-	(footprint "LOGO"
+	(footprint "Library:LOGO"
 		(locked yes)
 		(layer "F.Cu")
@@
 		)
 	)
-	(footprint "Capacitor_SMD:C_0402_1005Metric"
+	(footprint "Library:C_0402_1005Metric"
 		(locked yes)
 		(layer "F.Cu")
@@
 		)
 	)
-	(footprint "Capacitor_SMD:C_0402_1005Metric"
+	(footprint "Library:C_0402_1005Metric"
 		(locked yes)
 		(layer "F.Cu")
@@
 		)
 	)
-	(footprint "Capacitor_SMD:C_0402_1005Metric"
+	(footprint "Library:C_0402_1005Metric"
 		(locked yes)
 		(layer "F.Cu")
@@
 		)
 	)
-	(footprint "Capacitor_SMD:C_0402_1005Metric"
+	(footprint "Library:C_0402_1005Metric"
 		(locked yes)
 		(layer "F.Cu")
@@
 		)
 	)
-	(footprint "TestPoint:TestPoint_Pad_D1.0mm"
+	(footprint "Library:TestPoint_Pad_D1.0mm"
 		(locked yes)
 		(layer "F.Cu")
@@
 		)
 	)
-	(footprint "TestPoint:TestPoint_Pad_D1.0mm"
+	(footprint "Library:TestPoint_Pad_D1.0mm"
 		(locked yes)
 		(layer "F.Cu")
@@
 		)
 	)
-	(footprint "Capacitor_SMD:C_0402_1005Metric"
+	(footprint "Library:C_0402_1005Metric"
 		(locked yes)
 		(layer "F.Cu")
@@
 		)
 	)
-	(footprint "Resistor_SMD:R_0603_1608Metric"
+	(footprint "Library:R_0603_1608Metric"
 		(locked yes)
 		(layer "F.Cu")
@@
 		)
 	)
-	(footprint "U's Footprint Library:0896BM15E0025"
+	(footprint "Library:0896BM15E0025"
 		(locked yes)
 		(layer "F.Cu")
@@
 		)
 	)
-	(footprint "Capacitor_SMD:C_0402_1005Metric"
+	(footprint "Library:C_0402_1005Metric"
 		(locked yes)
 		(layer "F.Cu")
@@
 		)
 	)
-	(footprint "Resistor_SMD:R_0603_1608Metric"
+	(footprint "Library:R_0603_1608Metric"
 		(locked yes)
 		(layer "F.Cu")
@@
 		)
 	)
-	(footprint "Capacitor_SMD:C_0402_1005Metric"
+	(footprint "Library:C_0402_1005Metric"
 		(locked yes)
 		(layer "F.Cu")
@@
 		)
 	)
-	(footprint "Capacitor_SMD:C_0402_1005Metric"
+	(footprint "Library:C_0402_1005Metric"
 		(locked yes)
 		(layer "F.Cu")
@@
 		)
 	)
-	(footprint "Capacitor_SMD:C_0402_1005Metric"
+	(footprint "Library:C_0402_1005Metric"
 		(locked yes)
 		(layer "F.Cu")
@@
 		)
 	)
-	(footprint "Resistor_SMD:R_0603_1608Metric"
+	(footprint "Library:R_0603_1608Metric"
 		(locked yes)
 		(layer "F.Cu")
@@
 		)
 	)
-	(footprint "Package_TO_SOT_SMD:SOT-23-3"
+	(footprint "Library:SOT-23-3"
 		(locked yes)
 		(layer "F.Cu")
@@
 		)
 	)
-	(footprint "Capacitor_SMD:C_0402_1005Metric"
+	(footprint "Library:C_0402_1005Metric"
 		(locked yes)
 		(layer "F.Cu")
