File: AT86RF215 Breakout Board.kicad_sch (KiCad schematic)
At the start: 52 parts, among them J1 USB_C, J2 896 ISM, J3 GPIO, J4 2.4G ISM, J5 Molex 53748-0408, J6 Frontend GPIO, J7 SPI Header, U1 XC6206P332MR-G, U2 AT86RF215, X1 7L26002007

Commit message: added local symbol and footprint libs
Parts:
- B1: symbol U's Symbol Library:0896BM15E0025001E -> Library:0896BM15E0025001E
- B2: symbol U's Symbol Library:2450FB15A0050001E -> Library:2450FB15A0050001E
- C1, C10, C11, C12, C13, C14, C15, C16, C17, C18, C19, C2, C20, C21, C22, C3, C4, C5, C6, C7, C8, C9: symbol Device:C -> Library:C
- H1, H2, H3, H4: symbol Mechanical:MountingHole -> Library:MountingHole
- J1: symbol Connector:USB_C_Receptacle_PowerOnly_6P -> Library:USB_C_Receptacle_PowerOnly_6P
- J2, J4: symbol Connector:Conn_Coaxial -> Library:Conn_Coaxial
- J3, J6: symbol Connector_Generic:Conn_01x06 -> Library:Conn_01x06
- J5: symbol Connector_Generic:Conn_02x20_Odd_Even -> Library:Conn_02x20_Odd_Even
- J7: symbol U's Symbol Library:SPI_Header -> Library:SPI_Header
- JP1: symbol Jumper:SolderJumper_2_Bridged -> Library:SolderJumper_2_Bridged
- L1: symbol Device:L -> Library:L
- R1, R2, R3, R4, R5, R6, R7: symbol Device:R -> Library:R
- TP1, TP2, TP4, TP5: symbol Connector:TestPoint -> Library:TestPoint
- TP3: symbol Connector:TestPoint_2Pole -> Library:TestPoint_2Pole
- U1: symbol Regulator_Linear:XC6206PxxxMR -> Library:XC6206PxxxMR
- U2: symbol U's Symbol Library:AT86RF215 -> Library:AT86RF215
- X1: symbol U's Symbol Library:TXC-7L Series -> Library:TXC-7L Series
